File: kicad/lepetocontrol.kicad_pcb (KiCad board)
At the start: 2 copper layers, 100.2 x 116.5 mm, 145 parts, among them J1 1x05, J10 SENSE1, J11 SENSE2, J12 SENSE3, J13 SENSE4, J2 1x05, J3 USB_OTG, J4 Conn_01x05, J5 Conn_01x03, J6 Conn_01x05_Female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

Commit message: wip wip wip
kicad files updated to version 8
vfd added
Connections:
- net /mcu/~OLED_RES renamed /mcu/~{OLED_RES}
- net /mcu/~RESET renamed /mcu/~{RESET}
Other:
- net class Default removed
- board text added: "~{RST}"
- board text removed: "~RST"
