File: kicad/lepetocontrol.sch (KiCad schematic (older format))
At the start: 92 parts, among them J1 1x05, J2 1x05, Q1 BC817, Q2 BC817, Q3 BC817, Q4 BC817, Q5 BC817, Q6 BC817, Q7 BC817, Q8 BC817, U1 74HC595, U2 74HC595

Commit message: wip wip wip
kicad files updated to version 8
vfd added
Parts:
- D1, D10, D11, D12, D13, D14, D15, D17, D18, D19, D2, D20, D21, D22, D23, D24, D25, D26, D27, D28, D29, D3, D30, D31, D33, D34, D35, D36, D37, D38, D39, D4, D40, D41, D42, D43, D44, D45, D46, D47, D49, D5, D50, D51, D52, D53, D54, D55, D56, D57, D58, D59, D6, D60, D61, D62, D63, D7, D8, D9: symbol device:LED -> lepetocontrol-rescue:LED-device
- H1, H2, H3, H4: symbol mechanical:MountingHole -> lepetocontrol-rescue:MountingHole-mechanical
- J1, J2: symbol conn:Conn_01x05_Female -> lepetocontrol-rescue:Conn_01x05_Female-conn
- Q1, Q2, Q3, Q4, Q5, Q6, Q7, Q8: symbol transistors:BC817 -> lepetocontrol-rescue:BC817-transistors
- R1, R10, R11, R12, R13, R14, R15, R16, R2, R3, R4, R5, R6, R7, R8, R9: symbol device:R -> lepetocontrol-rescue:R-device
- U1, U2: symbol 74xx:74HC595 -> lepetocontrol-rescue:74HC595-74xx
