File: kicad/mcu.sch (KiCad schematic (older format))
At the start: 49 parts, among them J10 SENSE1, J11 SENSE2, J12 SENSE3, J13 SENSE4, J3 USB_OTG, J4 Conn_01x05, J5 Conn_01x03, J6 Conn_01x05_Female, J7 Conn_01x05_Female, J8 Conn_02x05_Odd_Even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

Commit message: wip wip wip
kicad files updated to version 8
vfd added
Parts:
- C1, C11, C13, C15, C2, C3, C4, C5, C6, C7, C8, C9: symbol device:C_Small -> lepetocontrol-rescue:C_Small-device
- C10: symbol device:CP -> lepetocontrol-rescue:CP-device
- H5, H6, H7, H8: symbol mechanical:MountingHole -> lepetocontrol-rescue:MountingHole-mechanical
- J10, J11, J12, J13: symbol conn:TEST_1P -> lepetocontrol-rescue:TEST_1P-conn
- J3: symbol conn:USB_OTG -> lepetocontrol-rescue:USB_OTG-conn
- J4: symbol conn:Conn_01x05 -> lepetocontrol-rescue:Conn_01x05-conn
- J5: symbol conn:Conn_01x03 -> lepetocontrol-rescue:Conn_01x03-conn
- J6, J7: symbol conn:Conn_01x05_Female -> lepetocontrol-rescue:Conn_01x05_Female-conn
- J8, J9: symbol conn:Conn_02x05_Odd_Even -> lepetocontrol-rescue:Conn_02x05_Odd_Even-conn
- R17, R18, R19, R20, R22: symbol device:R -> lepetocontrol-rescue:R-device
- SW1, SW2, SW3, SW4, SW5, SW6: symbol switches:SW_Push -> lepetocontrol-rescue:SW_Push-switches
- U3: symbol regul:LM1117-3.3 -> lepetocontrol-rescue:LM1117-3.3-regul
- U4: symbol stm32:STM32F103C4Tx -> lepetocontrol-rescue:STM32F103C4Tx-stm32
- U6: symbol 74xx:74HC595 -> lepetocontrol-rescue:74HC595-74xx
- U8: symbol 74xx:74HC4051 -> lepetocontrol-rescue:74HC4051-74xx
- Y1: symbol device:Crystal -> lepetocontrol-rescue:Crystal-device
